Commit message: add trajectory node. gripper joint not working yet

File: urdf/robots/reactor_description-grip.urdf (robot description, URDF)
Before this commit: robot reactor_description, 7 links, 6 joints
Joints:
- joint elbow_pitch: axis 0 1 0 -> 0 -1 0; limit lower=-3.141593 upper=0 effort=3.0 velocity=6.178465545 -> lower=-3.141593 upper=3.141593 effort=3.0 velocity=6.178465545
- joint shoulder_pitch: axis 0 1 0 -> 0 -1 0; limit lower=0 upper=3.141593 effort=3.0 velocity=6.178465545 -> lower=-3.141593 upper=3.141593 effort=3.0 velocity=6.178465545
- joint wrist_pitch: axis 0 1 0 -> 0 -1 0

Commit message: got gripper working

File: urdf/robots/reactor_description-grip.urdf (robot description, URDF)
Before this commit: robot reactor_description, 7 links, 6 joints
Joints:
- removed joint wrist_roll
- added joint wrist_yaw: type revolute, parent wrist_1, child wrist_2, origin xyz=0.071 0.00175 0 rpy=0 0 0, axis 1 0 0, limit lower=-3.141593 upper=3.141593 effort=1.5 velocity=6.178465545

File: urdf/robots/reactor_description.urdf (robot description, URDF)
Before this commit: robot reactor_description, 7 links, 6 joints
Joints:
- removed joint wrist_roll
- added joint wrist_yaw: type revolute, parent wrist_1, child wrist_2, origin xyz=0.071 0.00175 0 rpy=0 0 0, axis 1 0 0, limit lower=-3.141593 upper=3.141593 effort=1.5 velocity=6.178465545
- joint gripper_joint: axis 0 0 0 -> 1 0 0; limit (none) -> lower=-3.14 upper=3.14 effort=1.5 velocity=6.17; type fixed -> revolute
